Commit message: updated ball chase project

File: ball_chase/src/my_robot/urdf/my_robot.xacro (robot description, xacro)
@@ -161,5 +161,5 @@
     <visual>
       <geometry>
-        <mesh filename="package://my_robot/meshes/hokuyo.dae"/>
+        <mesh filename="package://my_robot/meshes/hokuyo.dae" />
       </geometry>
     </visual>
@@ -173,11 +173,11 @@
   <!-- Given components some color -->
   <gazebo reference="chassis">
-    <material>Gazebo/Green</material>
+    <material>Gazebo/Orange</material>
 	</gazebo>
   <gazebo reference="left_wheel">
-    <material>Gazebo/Orange</material>
+    <material>Gazebo/Blue</material>
 	</gazebo>
 	<gazebo reference="right_wheel">
-    <material>Gazebo/Orange</material>
+    <material>Gazebo/Blue</material>
 	</gazebo>
 	<gazebo reference="camera">
